Commit message: .

File: universal_robot/ur_description/urdf/left_arm_ur3_robot.urdf.xacro (robot description, xacro)
@@ -19,5 +19,5 @@
     <parent link="world" />
     <child link = "left_arm_base_link" />
-    <origin xyz="0.0 $(arg initial_position) 0.08" rpy="0.0 0.0 0.0" />
+    <origin xyz="0.0 0 0.08" rpy="0.0 0.0 0.0" />
   </joint>
 </robot>

File: universal_robot/ur_description/urdf/right_arm_ur3_robot.urdf.xacro (robot description, xacro)
@@ -15,9 +15,14 @@
     initial_position="$(arg initial_position)"
   />
+  <xacro:property name="yaml_file" value="$(find ur_description)/urdf/final_transform.yaml" />
+  <xacro:property name="transform" value="${load_yaml(yaml_file)}"/>
+  <xacro:property name="x" value="${transform['x']}" />
+  <xacro:property name="y" value="${transform['y']}" />
+  <xacro:property name="z" value="${transform['z']}" />
   <link name="world" />
   <joint name="world_joint" type="fixed">
     <parent link="world" />
     <child link = "right_arm_base_link" />
-    <origin xyz="0.0 $(arg initial_position) 0.08" rpy="0.0 0.0 0.0" />
+    <origin xyz="${x} ${y} ${z + 0.08}" rpy="0.0 0.0 0.0" />
   </joint>
 </robot>

File: universal_robot/ur_description/urdf/ur3gripper.urdf.xacro (robot description, xacro)
@@ -314,5 +314,5 @@
       <collision>
         <geometry>
-          <box size="0.01 0.01 213.0"/>
+          <box size="0.01 0.01 0.213"/>
         </geometry>
         <origin rpy="0 0 0" xyz="-0.01 0 0"/>
