Commit message: .

File: universal_robot/ur_description/urdf/ur3gripper.urdf.xacro (robot description, xacro)
@@ -316,5 +316,5 @@
           <box size="0.01 0.01 0.213"/>
         </geometry>
-        <origin rpy="0 0 0" xyz="-0.01 0 0"/>
+        <origin rpy="0 0 0" xyz="-0.01 0 0.1"/>
       </collision>
     </link>
